File: KiCad/GassTass/_saved_GassTass.sch (KiCad schematic (older format))
At the start: 94 parts, among them J1 EURO_PWR_2x5, J10 PJ301M-12, J11 PJ301M-12, J2 PJ301M-12, J3 PJ301M-12, J4 PJ301M-12, J5 PJ301M-12, J6 PJ301M-12, J7 PJ301M-12, J8 PJ301M-12, J9 PJ301M-12, Q1 2N3904, Q10 2N3904, Q11 2N3904, Q12 2N3904, Q13 2N3904, Q14 2N3904, Q15 2N3904, Q16 2N3904, Q17 2N3904, Q18 2N3904, Q19 2N3904, Q2 2N3904, Q3 2N3904, Q4 2N3904, Q5 2N3904, Q6 2N3904, Q7 2N3904, Q8 2N3904, Q9 2N3904, U1 Arduino_Nano_v3.x, U2 ATmega328P-PU

Commit message: redesigning pcb
Parts:
- removed D4: LED, LED_THT:LED_D3.0mm_FlatTop, symbol Device:LED
- removed J3: PJ301M-12, eurorack:PJ301M-12, symbol Eurorack:PJ301M-12
- removed Q5: 2N3904, Package_TO_SOT_THT:TO-92_Inline, symbol Transistor_BJT:2N3904
- removed R13: R_US, Resistor_THT:R_Axial_DIN0207_L6.3mm_D2.5mm_P10.16mm_Horizontal, symbol Device:R_US
Connections:
- wire segments 261 -> 255
Changed lines of the file:
@@
 	0    1    -1   0
 $EndComp
-$Comp
-L Transistor_BJT:2N3904 Q5
-U 1 1 5C7C5BC1
-P 3000 9200
-F 0 "Q5" V 3235 9200 50  0000 C CNN
-F 1 "2N3904" V 3326 9200 50  0000 C CNN
-F 2 "Package_TO_SOT_THT:TO-92_Inline" H 3200 9125 50  0001 L CIN
-F 3 "https://www.fairchildsemi.com/datasheets/2N/2N3904.pdf" H 3000 9200 50  0001 L CNN
-	1    3000 9200
-	0    1    1    0
-$EndComp
-$Comp
-L Eurorack:PJ301M-12 J3
-U 1 1 5C7C5BC7
-P 1650 9200
-F 0 "J3" H 1658 9575 50  0000 C CNN
-F 1 "PJ301M-12" H 1658 9484 50  0000 C CNN
-F 2 "eurorack:PJ301M-12" H 1650 9200 50  0001 C CNN
-F 3 "" H 1650 9200 50  0000 C CNN
-	1    1650 9200
-	1    0    0    -1
-$EndComp
-$Comp
-L Device:LED D4
-U 1 1 5C7C5BCD
-P 2750 9050
-F 0 "D4" H 2743 9266 50  0000 C CNN
-F 1 "LED" H 2743 9175 50  0000 C CNN
-F 2 "LED_THT:LED_D3.0mm_FlatTop" H 2750 9050 50  0001 C CNN
-F 3 "~" H 2750 9050 50  0001 C CNN
-	1    2750 9050
-	1    0    0    -1
-$EndComp
-$Comp
-L Device:R_US R13
-U 1 1 5C7C5BD3
-P 2350 9050
-F 0 "R13" H 2418 9096 50  0000 L CNN
-F 1 "R_US" H 2418 9005 50  0000 L CNN
-F 2 "Resistor_THT:R_Axial_DIN0207_L6.3mm_D2.5mm_P10.16mm_Horizontal" V 2390 9040 50  0001 C CNN
-F 3 "~" H 2350 9050 50  0001 C CNN
-	1    2350 9050
-	0    -1   -1   0
-$EndComp
-$Comp
-L power:+12V #PWR0105
-U 1 1 5C7C5BD9
-P 3200 9300
-F 0 "#PWR0105" H 3200 9150 50  0001 C CNN
-F 1 "+12V" V 3215 9428 50  0000 L CNN
-F 2 "" H 3200 9300 50  0001 C CNN
-F 3 "" H 3200 9300 50  0001 C CNN
-	1    3200 9300
-	0    1    -1   0
-$EndComp
-Wire Wire Line
-	3000 9000 2900 9000
-Wire Wire Line
-	2900 9000 2900 9050
-Wire Wire Line
-	2600 9050 2500 9050
-Wire Wire Line
-	2200 9050 2100 9050
-Wire Wire Line
-	2100 9300 2800 9300
-Wire Wire Line
-	2100 9200 2100 9050
-Connection ~ 2100 9050
-$Comp
-L power:GND #PWR0106
-U 1 1 5C7C5BE6
-P 2100 9200
-F 0 "#PWR0106" H 2100 8950 50  0001 C CNN
-F 1 "GND" V 2105 9072 50  0000 R CNN
-F 2 "" H 2100 9200 50  0001 C CNN
-F 3 "" H 2100 9200 50  0001 C CNN
-	1    2100 9200
-	0    -1   1    0
-$EndComp
-Connection ~ 2100 9200
 Text GLabel 1000 4500 1    50   Input ~ 0
 Tr1-in
