File: NTP/hw/NTP.sch (KiCad schematic (older format))
At the start: 95 parts, among them J1 PJ301M-12, J2 PJ301M-12, J3 PJ301M-12, J4 PJ301M-12, J5 PJ301M-12, J6 PJ301M-12, J7 PJ301M-12, J8 PJ301M-12, J9 PJ301M-12, Q1 2N3904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

Commit message: added exp
Parts:
- C1, C2: footprint Capacitor_SMD:CP_Elec_6.3x5.4 -> Capacitor_SMD:CP_Elec_5x5.3
Changed lines of the file:
@@
 F 0 "C2" H 7791 6146 50  0000 L CNN
 F 1 "470n" H 7791 6055 50  0000 L CNN
-F 2 "Capacitor_SMD:CP_Elec_6.3x5.4" H 7700 6100 50  0001 C CNN
+F 2 "Capacitor_SMD:CP_Elec_5x5.3" H 7700 6100 50  0001 C CNN
 F 3 "~" H 7700 6100 50  0001 C CNN
 F 4 "" H 7700 6100 50  0001 C CNN "Field4"
@@
 F 0 "C1" H 7791 5846 50  0000 L CNN
 F 1 "470n" H 7791 5755 50  0000 L CNN
-F 2 "Capacitor_SMD:CP_Elec_6.3x5.4" H 7700 5800 50  0001 C CNN
+F 2 "Capacitor_SMD:CP_Elec_5x5.3" H 7700 5800 50  0001 C CNN
 F 3 "~" H 7700 5800 50  0001 C CNN
 F 4 "" H 7700 5800 50  0001 C CNN "Field4"
