File: NTP/hw/NTPv02.kicad_pcb (KiCad board)
At the start: 2 copper layers, 39.4 x 106.7 mm, 68 parts, among them J1 PJ301M-12, J2 PJ301M-12, J3 PJ301M-12, J4 PJ301M-12, J5 PJ301M-12, J6 PJ301M-12, J7 PJ301M-12, J8 PJ301M-12, J9 PJ301M-12, Q1 2N3904, Q2 2N3904, Q3 2N3904, Q4 2N3904, Q5 2N3904, Q6 2N3904, Q7 2N3904, Q8 2N3904, Q9 2N3904

Commit message: locked panel
Parts:
- Q1, Q2, Q3, Q4, Q5, Q6, Q7, Q8, Q9, R1, R10, R11, R12, R13, R14, R15, R16, R17, R18, R19, R2, R20, R21, R22, R23, R24, R25, R26, R27, R3, R4, R5, R6, R7, R8, R9: moved to B.Cu
- moved Q3 138.9 mm to (104.1, 126.4), turned to 180 degrees
- moved Q6 133.2 mm to (104.1, 139.7), turned to 180 degrees
- moved Q2 127.7 mm to (92.1, 126.4), turned to 180 degrees
- moved Q9 126.9 mm to (104.1, 150.5), turned to 180 degrees
- moved Q5 121.2 mm to (92.1, 139.7), turned to 180 degrees
- moved Q1 117.0 mm to (80.0, 126.4), turned to 180 degrees
- moved Q8 114.6 mm to (92.1, 150.5), turned to 180 degrees
- moved Q4 109.9 mm to (80.0, 139.7), turned to 180 degrees
- moved Q7 102.5 mm to (80.0, 150.5), turned to 180 degrees
- moved R10 73.9 mm to (81.3, 131.1), turned to 90 degrees
- moved R22 73.3 mm to (81.3, 155.2), turned to 90 degrees
- moved R16 72.1 mm to (81.3, 135.0), turned to 270 degrees
- moved R1 70.3 mm to (78.7, 131.1), turned to 90 degrees
- moved R7 69.6 mm to (78.7, 155.2), turned to 90 degrees
- moved R4 68.3 mm to (78.7, 135.0), turned to 270 degrees
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Routing:
- net GND: track 0.00 -> 367.6 mm, vias 0 -> 2
- net 5V: track 0.00 -> 212.6 mm, vias 0 -> 1
- net Tr9: track 0.00 -> 128.2 mm, vias 0 -> 3
- net Tr8: track 0.00 -> 124.0 mm, vias 0 -> 7
- net Tr6: track 0.00 -> 99.7 mm, vias 0 -> 7
- net Tr3: track 0.00 -> 89.1 mm, vias 0 -> 4
- net Tr7: track 0.00 -> 81.6 mm, vias 0 -> 1
- net Tr5: track 0.00 -> 61.5 mm, vias 0 -> 3
- net Tr4: track 0.00 -> 50.7 mm, vias 0 -> 2
- net Tr2: track 0.00 -> 45.8 mm, vias 0 -> 3
- net SDA: track 0.00 -> 42.0 mm, vias 0 -> 2
- net SDC: track 0.00 -> 37.0 mm, vias 0 -> 2
- net Tr1: track 0.00 -> 35.0 mm
- net 12V: track 0.00 -> 19.6 mm, vias 0 -> 1
- net Net-(D10-Pad1): track 0.00 -> 15.9 mm
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Other:
- outline, holes or cut-outs redrawn

Commit message: ok
Parts:
- H2: value PIN_HEADER_2x8 -> POWER
- moved H1 22.9 mm to (72.4, 73.7)
- moved R23 1.49 mm to (82.8, 111.1)
- moved D7 1.42 mm to (83.8, 113.0)
- moved D9 1.42 mm to (95.2, 113.0)
- moved R27 1.36 mm to (94.2, 111.1)
- moved D8 1.27 mm to (89.5, 113.0)
- moved R25 1.27 mm to (88.7, 111.1)
- moved R17 1.01 mm to (82.8, 105.4)
- moved D4 0.90 mm to (83.8, 107.3)
- moved D6 0.90 mm to (95.2, 107.3)
- moved R21 0.90 mm to (94.4, 105.4)
- moved D1 0.64 mm to (83.8, 101.6)
- moved D3 0.64 mm to (95.2, 101.6)
- moved R11 0.64 mm to (82.9, 99.7)
- moved D5 0.63 mm to (89.5, 107.3)
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Routing:
- net GND: track 367.6 -> 318.7 mm, vias 2 -> 7
- net 5V: track 212.6 -> 255.9 mm, vias 1 -> 11
- net Tr4: track 50.7 -> 82.7 mm, vias 2 -> 3
- net Tr1: track 35.0 -> 66.9 mm, vias 0 -> 2
- net Tr5: track 61.5 -> 86.9 mm
- net Tr7: track 81.6 -> 103.1 mm, vias 1 -> 3
- net Tr2: track 45.8 -> 64.9 mm, vias 3 -> 2
- net Tr3: track 89.1 -> 76.0 mm, vias 4 -> 2
- net Tr8: track 124.0 -> 131.3 mm, vias 7 -> 8
- net Tr9: track 128.2 -> 121.6 mm, vias 3 -> 5
- net SDC: track 37.0 -> 43.2 mm, vias 2 -> 1
- net Net-(A1-Pad18): track 15.6 -> 21.6 mm, vias 0 -> 1
- net Net-(D10-Pad1): track 15.9 -> 20.9 mm, vias 0 -> 2
- net Net-(A1-Pad19): track 12.0 -> 16.5 mm, vias 0 -> 1
- net Tr6: track 99.7 -> 104.0 mm, vias 7 -> 2
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- added copper zone on B.Cu, net (none)
- added copper zone on F.Cu, net GND
Other:
- outline, holes or cut-outs redrawn
- board text added: "SysAdm - NTP"

Commit message: added panel
Parts:
- added ?: , , F.Cu at (102.9, 54.0)
Changed lines of the file:
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@@
-(kicad_pcb (version 20171130) (host pcbnew "(5.1.0)-1")
+(kicad_pcb (version 20171130) (host pcbnew "(5.1.2)-1")
   (general
     (thickness 1.6)
-    (drawings 15)
+    (drawings 16)
     (tracks 518)
     (zones 0)
-    (modules 68)
+    (modules 69)
     (nets 67)
   )
   (page A4)
   (layers
-    (0 F.Cu signal)
-    (31 B.Cu signal)
-    (32 B.Adhes user)
-    (33 F.Adhes user)
-    (34 B.Paste user)
-    (35 F.Paste user)
-    (36 B.SilkS user)
-    (37 F.SilkS user)
-    (38 B.Mask user)
-    (39 F.Mask user)
-    (40 Dwgs.User user)
-    (41 Cmts.User user)
-    (42 Eco1.User user)
-    (43 Eco2.User user)
+    (0 F.Cu signal hide)
+    (31 B.Cu signal hide)
+    (32 B.Adhes user hide)
+    (33 F.Adhes user hide)
+    (34 B.Paste user hide)
+    (35 F.Paste user hide)
+    (36 B.SilkS user hide)
+    (37 F.SilkS user hide)
+    (38 B.Mask user hide)
+    (39 F.Mask user hide)
+    (40 Dwgs.User user hide)
+    (41 Cmts.User user hide)
+    (42 Eco1.User user hide)
+    (43 Eco2.User user hide)
     (44 Edge.Cuts user)
-    (45 Margin user)
-    (46 B.CrtYd user)
-    (47 F.CrtYd user)
-    (48 B.Fab user)
-    (49 F.Fab user)
+    (45 Margin user hide)
+    (46 B.CrtYd user hide)
+    (47 F.CrtYd user hide)
+    (48 B.Fab user hide)
+    (49 F.Fab user hide)
   )
   (setup
@@
     (add_net Tr9)
   )
+  (module "" (layer F.Cu)
+    (at 102.87 53.975)
+    (fp_text reference "" (at 90.805 74.93) (layer F.SilkS)
+      (effects (font (size 1.27 1.27) (thickness 0.15)))
+    )
+    (fp_text value "" (at 90.805 74.93) (layer F.SilkS)
+      (effects (font (size 1.27 1.27) (thickness 0.15)))
+    )
+    (fp_text user ------ (at 0 -0.635) (layer B.Mask)
+      (effects (font (size 1 1) (thickness 0.25)) (justify mirror))
+    )
+  )
   (module Potentiometer_THT:Potentiometer_Alpha_RD901F-40-00D_Single_Vertical (layer F.Cu)
     (at 90.805 74.93 270)
@@
     (descr "Through hole straight pin header, 2x08, 2.54mm pitch, double rows")
     (tags "Through hole pin header THT 2x08 2.54mm double row")
-    (fp_text reference H2 (at 4.445 -8.89 90) (layer B.SilkS)
+    (fp_text reference H2 (at -1.905 -8.89 90) (layer B.SilkS)
       (effects (font (size 1 1) (thickness 0.15)) (justify mirror))
     )
@@
     (fp_line (start 3.81 1.27) (end 3.81 -19.05) (layer B.Fab) (width 0.1))
     (fp_line (start 0 1.27) (end 3.81 1.27) (layer B.Fab) (width 0.1))
-    (fp_text user POWER (at 1.27 3.81 180) (layer B.SilkS)
+    (fp_text user POWER (at 1.27 3.175 180) (layer B.SilkS)
+      (effects (font (size 1 1) (thickness 0.15)) (justify mirror))
+    )
+    (fp_text user ------ (at 1.27 1.905 180) (layer B.Mask)
+      (effects (font (size 1 1) (thickness 0.25)) (justify mirror))
+    )
+    (fp_text user -12v (at 5.715 0 180) (layer B.SilkS)
+      (effects (font (size 1 1) (thickness 0.15)) (justify mirror))
+    )
+    (fp_text user 12v (at 5.715 -10.16 180) (layer B.SilkS)
       (effects (font (size 1 1) (thickness 0.15)) (justify mirror))
     )
-    (fp_text user RED (at 1.27 2.54 180) (layer B.SilkS)
+    (fp_text user 5v (at 5.08 -12.7 180) (layer B.SilkS)
       (effects (font (size 1 1) (thickness 0.15)) (justify mirror))
     )
@@
     )
   )
-  (gr_text "SysAdm - NTP" (at 72.39 96.52 90) (layer B.SilkS)
+  (gr_text "SysAdm - NTP" (at 72.39 97.79 90) (layer F.Mask)
+    (effects (font (size 3 3) (thickness 0.5)))
+  )
+  (gr_text "SysAdm - NTP" (at 72.39 96.52 90) (layer B.Mask)
     (effects (font (size 3 3) (thickness 0.5)) (justify mirror))
   )
@@
       )
     )
+  )
+  (zone (net 0) (net_name "") (layer F.Cu) (hatch edge 0.508)
+    (connect_pads (clearance 0.508))
+    (min_thickness 0.254)
+    (keepout (tracks allowed) (vias allowed) (copperpour not_allowed))
+    (fill (arc_segments 32) (thermal_gap 0.508) (thermal_bridge_width 0.508))
+    (polygon
+      (pts
+        (xy 69.215 120.65) (xy 74.93 120.65) (xy 74.93 120.015) (xy 75.565 119.38) (xy 76.835 119.38)
+        (xy 81.915 114.3) (xy 80.01 113.665) (xy 80.645 111.76) (xy 82.55 111.76) (xy 82.55 83.82)
+        (xy 80.01 80.01) (xy 80.01 54.61) (xy 74.93 54.61) (xy 74.93 58.42) (xy 69.215 58.42)
+      )
+    )
