File: NTP-exp/NTP-exp/NTP-exp.kicad_pcb (KiCad board)
At the start: 2 copper layers, 67 parts, among them J1 PJ301M-12, J10 PJ301M-12, J11 PJ301M-12, J12 PJ301M-12, J13 PJ301M-12, J14 PJ301M-12, J15 PJ301M-12, J16 PJ301M-12, J17 PJ301M-12, J18 PJ301M-12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

Commit message: designing
Parts:
- removed D4, D5, D6, D7: LED, LED_THT:LED_D3.0mm_FlatTop
- removed J15, J16, J17, J18: PJ301M-12, eurorack:PJ301M-12
- removed the R10 at (162.0, 51.5)
- removed R23, R24, R25, R28, R29, R30, R33, R34: 51, Resistor_SMD:R_0805_2012Metric_Pad1.15x1.40mm_HandSolder
- removed R26, R31: 10m, Resistor_SMD:R_0805_2012Metric_Pad1.15x1.40mm_HandSolder
- removed R27, R32: 1k, Resistor_SMD:R_0805_2012Metric_Pad1.15x1.40mm_HandSolder
- removed the R7 at (134.6, 129.2)
- removed the R8 at (147.0, 51.5)
- removed the R9 at (147.0, 46.5)
- removed the U2 at (143.0, 43.5)
- removed U6, U7: TL074, Package_DIP:DIP-14_W7.62mm_Socket
- added R11: 51, Resistor_SMD:R_0805_2012Metric_Pad1.15x1.40mm_HandSolder, F.Cu at (133.6, 88.2)
- added R12: 51, Resistor_SMD:R_0805_2012Metric_Pad1.15x1.40mm_HandSolder, F.Cu at (184.6, 48.2)
- added R13: 51, Resistor_SMD:R_0805_2012Metric_Pad1.15x1.40mm_HandSolder, F.Cu at (128.8, 88.2)
- added R14: 1k, Resistor_SMD:R_0805_2012Metric_Pad1.15x1.40mm_HandSolder, F.Cu at (133.6, 85.3)
- added U3: TL074, Package_DIP:DIP-14_W7.62mm_Socket, F.Cu at (120.2, 48.9)
- R1: value 51 -> 1k; moved to F.Cu
- R15: value 51 -> 10m
- R16, R21: value 10m -> 51
- R17, R22: value 1k -> 51
- R3: value 1k -> 51; moved to F.Cu
- R4, R5, U1: moved to F.Cu
- moved J9 113.0 mm to (156.8, 53.5)
- moved J12 103.2 mm to (163.8, 82.8)
- moved J11 102.1 mm to (153.6, 82.8)
- moved R21 97.4 mm to (124.1, 87.9)
- moved R19 92.4 mm to (118.2, 90.8)
- moved J7 90.0 mm to (156.8, 68.2)
- moved J8 88.6 mm to (166.9, 68.2)
- moved R22 88.2 mm to (119.3, 87.9)
- moved J14 86.2 mm to (173.9, 82.8)
- moved J13 85.4 mm to (177.1, 68.2)
- moved J10 84.0 mm to (177.1, 53.5)
- moved R20 81.5 mm to (128.8, 85.3)
- moved R1 80.5 mm to (108.7, 92.8)
- moved R17 75.5 mm to (131.1, 82.3)
- moved R4 75.2 mm to (123.0, 90.8)
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- renumbered R14 to R10, R11 to R7, R12 to R8, R13 to R9, U3 to U2
Connections:
- R1 pad 1: Net-(R1-Pad1) -> Net-(D1-Pad1)
- R1 pad 2: Net-(J1-Pad3) -> GND
- R15 pad 1: Net-(R15-Pad1) -> STr1
- R15 pad 2: Net-(J7-Pad3) -> GND
- R16 pad 1: GND -> Net-(R16-Pad1)
- R16 pad 2: STr3 -> Net-(J8-Pad3)
- R17 pad 1: Net-(D4-Pad2) -> Net-(R17-Pad1)
- R17 pad 2: GND -> Net-(J9-Pad3)
- R18 pad 2: Net-(J8-Pad3) -> Net-(J10-Pad3)
- R19 pad 2: Net-(J9-Pad3) -> Net-(J11-Pad3)
- R2 pad 1: GND -> STr1
- R2 pad 2: STr1 -> GND
- R20 pad 2: Net-(J10-Pad3) -> Net-(J12-Pad3)
- R21 pad 1: GND -> Net-(R21-Pad1)
- R21 pad 2: STr4 -> Net-(J13-Pad3)
- R22 pad 1: Net-(D5-Pad2) -> Net-(R22-Pad1)
- R22 pad 2: GND -> Net-(J14-Pad3)
- R3 pad 1: Net-(D1-Pad2) -> Net-(R3-Pad1)
- R3 pad 2: GND -> Net-(J1-Pad3)
- U1 pad 1: Net-(R1-Pad1) -> Net-(D1-Pad2)
- U1 pad 13: Net-(D1-Pad2) -> Net-(R5-Pad1)
- U1 pad 14: Net-(D1-Pad1) -> Net-(R5-Pad1)
- U1 pad 2: Net-(R1-Pad1) -> Net-(D1-Pad1)
- U1 pad 6: Net-(R4-Pad1) -> Net-(R3-Pad1)
- U1 pad 7: Net-(R4-Pad1) -> Net-(R3-Pad1)
- U1 pad 8: Net-(R5-Pad1) -> Net-(R4-Pad1)
- U1 pad 9: Net-(R5-Pad1) -> Net-(R4-Pad1)
- U4 pad 1: Net-(R15-Pad1) -> Net-(D3-Pad2)
- U4 pad 10: STr3 -> STr1
- U4 pad 11: (no net) -> GND
- U4 pad 12: STr3 -> STr1
- U4 pad 13: Net-(D4-Pad2) -> Net-(R18-Pad1)
- U4 pad 14: Net-(D4-Pad1) -> Net-(R18-Pad1)
- U4 pad 2: Net-(R15-Pad1) -> Net-(D3-Pad1)
- U4 pad 3: STr3 -> STr1
- U4 pad 4: (no net) -> 5V
- U4 pad 5: STr3 -> STr1
- U4 pad 6: Net-(R18-Pad1) -> Net-(R16-Pad1)
- U4 pad 7: Net-(R18-Pad1) -> Net-(R16-Pad1)
- U4 pad 8: Net-(R19-Pad1) -> Net-(R17-Pad1)
- U4 pad 9: Net-(R19-Pad1) -> Net-(R17-Pad1)
- U5 pad 1: Net-(R20-Pad1) -> Net-(R19-Pad1)
- U5 pad 10: STr4 -> STr1
- U5 pad 11: (no net) -> GND
- U5 pad 12: STr4 -> STr1
- U5 pad 13: Net-(D5-Pad2) -> Net-(R22-Pad1)
- U5 pad 14: Net-(D5-Pad1) -> Net-(R22-Pad1)
- U5 pad 2: Net-(R20-Pad1) -> Net-(R19-Pad1)
- U5 pad 3: STr4 -> STr1
- U5 pad 4: (no net) -> 5V
- U5 pad 5: STr4 -> STr1
- U5 pad 6: Net-(R23-Pad1) -> Net-(R20-Pad1)
- U5 pad 7: Net-(R23-Pad1) -> Net-(R20-Pad1)
- U5 pad 8: Net-(R24-Pad1) -> Net-(R21-Pad1)
- U5 pad 9: Net-(R24-Pad1) -> Net-(R21-Pad1)
