File: MLT/MLT.sch (KiCad schematic (older format))
At the start: 44 parts, among them J1 PJ301M-12, J10 PJ301M-12, J11 PJ301M-12, J12 PJ301M-12, J2 PJ301M-12, J3 PJ301M-12, J4 PJ301M-12, J5 PJ301M-12, J6 PJ301M-12, J7 PJ301M-12, J8 PJ301M-12, J9 PJ301M-12, U1 TL074, U2 TL074, U3 TL074

Commit message: ok
Parts:
- renumbered C5 to C2, C2 to C3, C6 to C4, C3 to C5, C7 to C6, C4 to C7, D4 to D3, D5 to D4, D3 to D5, J10 to J1, J3 to J10, J6 to J11, J9 to J12, J1 to J2, J4 to J3, J7 to J4, J11 to J5, J2 to J6, J5 to J7, J12 to J9, R4 to R1, R11 to R10, R6 to R11, R15 to R12, R3 to R13, R9 to R14, R12 to R15, R13 to R2, R1 to R3, R7 to R4, R10 to R5, R5 to R6, R14 to R7, R2 to R8, R8 to R9
Connections:
- net GND: now also J1.1, J9.1; no longer J1.3, J9.3
- net at R1.1, U1.10 (+), U1.12 (+)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: now also J1.3; no longer J1.1
- net at R11.1, U3.10 (+), U3.12 (+)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: now also J9.3; no longer J9.1
Other:
- moved on the sheet: R1, R11
