File: takt/ex/takt-exp-panel.kicad_pcb (KiCad board)
At the start: 2 copper layers, 40.3 x 128.5 mm, 55 parts, among them J1 PJ301M-12, J2 PJ301M-12, J3 PJ301M-12, J4 PJ301M-12, J5 PJ301M-12, J6 PJ301M-12, J7 PJ301M-12, J8 PJ301M-12, J9 PJ301M-12, Q1 2N3904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

Commit message: exp traced
Parts:
- turned J1 to 180 degrees
- turned J2 to 0 degrees
- turned J3 to 180 degrees
- turned J4 to 180 degrees
- turned J5 to 0 degrees
- turned J6 to 180 degrees
- turned J7 to 180 degrees
- turned J8 to 0 degrees
- turned J9 to 180 degrees
Other:
- board size 40.3 x 128.5 mm -> 147.8 x 128.5 mm

Commit message: exp panel
Parts:
- removed D1: CC56-12CGKWA, Display_7Segment:AFF_2x7SEG-DIGIT_10mm
- removed D2, D3, D4, D5, D6, D7: LED, LED_THT:LED_D3.0mm_FlatTop
- removed H1: Expander, Connector_PinHeader_2.54mm:PinHeader_2x08_P2.54mm_Vertical
- removed J1, J2, J3, J4, J5, J6, J7, J8, J9: PJ301M-12, eurorack:PJ301M-12
- removed Q1, Q2, Q3: 2N3904, Package_TO_SOT_SMD:SOT-23
- removed R1, R2, R26, R27, R28, R3, R4: 200, Resistor_SMD:R_0603_1608Metric_Pad1.05x0.95mm_HandSolder
- removed R10, R11, R12, R13, R5, R6, R7, R8, R9: 51, Resistor_SMD:R_0805_2012Metric_Pad1.15x1.40mm_HandSolder
- removed R14, R15, R16: 6.8k, Resistor_SMD:R_0603_1608Metric_Pad1.05x0.95mm_HandSolder
- removed R17, R18, R19: 2.2k, Resistor_SMD:R_0603_1608Metric_Pad1.05x0.95mm_HandSolder
- removed R20, R21, R22: 10m, Resistor_SMD:R_0805_2012Metric_Pad1.15x1.40mm_HandSolder
- removed R23, R24, R25: 1k, Resistor_SMD:R_0805_2012Metric_Pad1.15x1.40mm_HandSolder
- removed SW1, SW2, SW3: SW_SP3T, Button_Switch_THT:SW_CuK_JS202011CQN_DPDT_Straight
- removed U1, U2, U3: TL074, Package_DIP:DIP-14_W7.62mm_Socket
- removed U4: ATmega328P-PU, Package_DIP:DIP-28_W7.62mm_Socket
Other:
- board size 147.8 x 128.5 mm -> 40.3 x 128.5 mm
- board text added: "1/32 1/9 1/5"
- board text added: "1/8 1/3 1/16"
- board text added: "4/4 1/4 2/4"
- board text added: "rot"
- board text added: "takt-exp"
