File: rør/MLT.sch (KiCad schematic (older format))
At the start: 44 parts, among them J1 PJ301M-12, J10 PJ301M-12, J11 PJ301M-12, J12 PJ301M-12, J2 PJ301M-12, J3 PJ301M-12, J4 PJ301M-12, J5 PJ301M-12, J6 PJ301M-12, J7 PJ301M-12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

Commit message: mlt update
Parts:
- H1: symbol eurocad:PIN_HEADER_2x5 -> MLT-rescue:PIN_HEADER_2x5-eurocad
- J1, J10, J11, J12, J2, J3, J4, J5, J6, J7, J8, J9: footprint eurocad:PJ301M-12 -> eurorack:PJ301M-12; symbol eurocad:PJ301M-12 -> MLT-rescue:PJ301M-12-eurocad
- U1, U2, U3: footprint Package_DIP:DIP-14_W8.89mm_SMDSocket_LongPads -> Package_DIP:SMDIP-14_W9.53mm
Changed lines of the file:
@@
 EESchema Schematic File Version 4
+LIBS:MLT-cache
 EELAYER 29 0
 EELAYER END
@@
 F 0 "U1" H 2300 2467 50  0000 C CNN
 F 1 "TL074" H 2300 2376 50  0000 C CNN
-F 2 "Package_DIP:DIP-14_W8.89mm_SMDSocket_LongPads" H 2250 2200 50  0001 C CNN
+F 2 "Package_DIP:SMDIP-14_W9.53mm" H 2250 2200 50  0001 C CNN
 F 3 "http://www.ti.com/lit/ds/symlink/tl071.pdf" H 2350 2300 50  0001 C CNN
 	1    2300 2100
@@
 F 0 "U1" H 2300 2967 50  0000 C CNN
 F 1 "TL074" H 2300 2876 50  0000 C CNN
-F 2 "Package_DIP:DIP-14_W8.89mm_SMDSocket_LongPads" H 2250 2700 50  0001 C CNN
+F 2 "Package_DIP:SMDIP-14_W9.53mm" H 2250 2700 50  0001 C CNN
 F 3 "http://www.ti.com/lit/ds/symlink/tl071.pdf" H 2350 2800 50  0001 C CNN
 	2    2300 2600
@@
 F 0 "U1" H 2300 3467 50  0000 C CNN
 F 1 "TL074" H 2300 3376 50  0000 C CNN
-F 2 "Package_DIP:DIP-14_W8.89mm_SMDSocket_LongPads" H 2250 3200 50  0001 C CNN
+F 2 "Package_DIP:SMDIP-14_W9.53mm" H 2250 3200 50  0001 C CNN
 F 3 "http://www.ti.com/lit/ds/symlink/tl071.pdf" H 2350 3300 50  0001 C CNN
 	3    2300 3100
@@
 F 0 "U1" H 2300 3967 50  0000 C CNN
 F 1 "TL074" H 2300 3876 50  0000 C CNN
-F 2 "Package_DIP:DIP-14_W8.89mm_SMDSocket_LongPads" H 2250 3700 50  0001 C CNN
+F 2 "Package_DIP:SMDIP-14_W9.53mm" H 2250 3700 50  0001 C CNN
 F 3 "http://www.ti.com/lit/ds/symlink/tl071.pdf" H 2350 3800 50  0001 C CNN
 	4    2300 3600
@@
 Connection ~ 1950 2000
 $Comp
-L eurocad:PJ301M-12 J1
+L MLT-rescue:PJ301M-12-eurocad J1
 U 1 1 5CD409F7
 P 1600 3400
 F 0 "J1" V 1654 3638 50  0000 L CNN
 F 1 "PJ301M-12" V 1563 3638 50  0000 L CNN
-F 2 "eurocad:PJ301M-12" H 1600 3400 50  0001 C CNN
+F 2 "eurorack:PJ301M-12" H 1600 3400 50  0001 C CNN
 F 3 "" H 1600 3400 50  0000 C CNN
 	1    1600 3400
@@
 Connection ~ 2600 3100
 $Comp
-L eurocad:PJ301M-12 J2
+L MLT-rescue:PJ301M-12-eurocad J2
 U 1 1 5CD505AA
 P 3350 2200
 F 0 "J2" H 2872 2184 50  0000 R CNN
 F 1 "PJ301M-12" H 2872 2275 50  0000 R CNN
-F 2 "eurocad:PJ301M-12" H 3350 2200 50  0001 C CNN
+F 2 "eurorack:PJ301M-12" H 3350 2200 50  0001 C CNN
 F 3 "" H 3350 2200 50  0000 C CNN
 	1    3350 2200
@@
 $EndComp
 $Comp
-L eurocad:PJ301M-12 J3
+L MLT-rescue:PJ301M-12-eurocad J3
 U 1 1 5CD549DA
 P 3350 2700
 F 0 "J3" H 2872 2684 50  0000 R CNN
 F 1 "PJ301M-12" H 2872 2775 50  0000 R CNN
-F 2 "eurocad:PJ301M-12" H 3350 2700 50  0001 C CNN
+F 2 "eurorack:PJ301M-12" H 3350 2700 50  0001 C CNN
 F 3 "" H 3350 2700 50  0000 C CNN
 	1    3350 2700
@@
 $EndComp
 $Comp
-L eurocad:PJ301M-12 J4
+L MLT-rescue:PJ301M-12-eurocad J4
 U 1 1 5CD54EDE
 P 3350 3200
 F 0 "J4" H 2872 3184 50  0000 R CNN
 F 1 "PJ301M-12" H 2872 3275 50  0000 R CNN
-F 2 "eurocad:PJ301M-12" H 3350 3200 50  0001 C CNN
+F 2 "eurorack:PJ301M-12" H 3350 3200 50  0001 C CNN
 F 3 "" H 3350 3200 50  0000 C CNN
 	1    3350 3200
@@
 $EndComp
 $Comp
-L eurocad:PIN_HEADER_2x5 H1
+L MLT-rescue:PIN_HEADER_2x5-eurocad H1
 U 1 1 5CD58F42
 P 6350 5750
@@
 F 0 "U2" H 5300 2467 50  0000 C CNN
 F 1 "TL074" H 5300 2376 50  0000 C CNN
-F 2 "Package_DIP:DIP-14_W8.89mm_SMDSocket_LongPads" H 5250 2200 50  0001 C CNN
+F 2 "Package_DIP:SMDIP-14_W9.53mm" H 5250 2200 50  0001 C CNN
 F 3 "http://www.ti.com/lit/ds/symlink/tl071.pdf" H 5350 2300 50  0001 C CNN
 	1    5300 2100
@@
 F 0 "U2" H 5300 2967 50  0000 C CNN
 F 1 "TL074" H 5300 2876 50  0000 C CNN
-F 2 "Package_DIP:DIP-14_W8.89mm_SMDSocket_LongPads" H 5250 2700 50  0001 C CNN
+F 2 "Package_DIP:SMDIP-14_W9.53mm" H 5250 2700 50  0001 C CNN
 F 3 "http://www.ti.com/lit/ds/symlink/tl071.pdf" H 5350 2800 50  0001 C CNN
 	2    5300 2600
@@
 F 0 "U2" H 5300 3467 50  0000 C CNN
 F 1 "TL074" H 5300 3376 50  0000 C CNN
-F 2 "Package_DIP:DIP-14_W8.89mm_SMDSocket_LongPads" H 5250 3200 50  0001 C CNN
+F 2 "Package_DIP:SMDIP-14_W9.53mm" H 5250 3200 50  0001 C CNN
 F 3 "http://www.ti.com/lit/ds/symlink/tl071.pdf" H 5350 3300 50  0001 C CNN
 	3    5300 3100
@@
 F 0 "U2" H 5300 3967 50  0000 C CNN
 F 1 "TL074" H 5300 3876 50  0000 C CNN
-F 2 "Package_DIP:DIP-14_W8.89mm_SMDSocket_LongPads" H 5250 3700 50  0001 C CNN
+F 2 "Package_DIP:SMDIP-14_W9.53mm" H 5250 3700 50  0001 C CNN
 F 3 "http://www.ti.com/lit/ds/symlink/tl071.pdf" H 5350 3800 50  0001 C CNN
 	4    5300 3600
@@
 Connection ~ 4950 2000
 $Comp
-L eurocad:PJ301M-12 J5
+L MLT-rescue:PJ301M-12-eurocad J5
 U 1 1 5CDC1AA2
 P 4650 3400
 F 0 "J5" V 4704 3222 50  0000 R CNN
 F 1 "PJ301M-12" V 4613 3222 50  0000 R CNN
-F 2 "eurocad:PJ301M-12" H 4650 3400 50  0001 C CNN
+F 2 "eurorack:PJ301M-12" H 4650 3400 50  0001 C CNN
 F 3 "" H 4650 3400 50  0000 C CNN
 	1    4650 3400
@@
 Connection ~ 5600 3100
 $Comp
-L eurocad:PJ301M-12 J6
+L MLT-rescue:PJ301M-12-eurocad J6
 U 1 1 5CDC1AD7
 P 6350 2200
 F 0 "J6" H 5872 2184 50  0000 R CNN
 F 1 "PJ301M-12" H 5872 2275 50  0000 R CNN
-F 2 "eurocad:PJ301M-12" H 6350 2200 50  0001 C CNN
+F 2 "eurorack:PJ301M-12" H 6350 2200 50  0001 C CNN
 F 3 "" H 6350 2200 50  0000 C CNN
 	1    6350 2200
@@
 $EndComp
 $Comp
-L eurocad:PJ301M-12 J7
+L MLT-rescue:PJ301M-12-eurocad J7
 U 1 1 5CDC1ADD
 P 6350 2700
 F 0 "J7" H 5872 2684 50  0000 R CNN
 F 1 "PJ301M-12" H 5872 2775 50  0000 R CNN
-F 2 "eurocad:PJ301M-12" H 6350 2700 50  0001 C CNN
+F 2 "eurorack:PJ301M-12" H 6350 2700 50  0001 C CNN
 F 3 "" H 6350 2700 50  0000 C CNN
 	1    6350 2700
@@
 $EndComp
 $Comp
-L eurocad:PJ301M-12 J8
+L MLT-rescue:PJ301M-12-eurocad J8
 U 1 1 5CDC1AE3
 P 6350 3200
 F 0 "J8" H 5872 3184 50  0000 R CNN
 F 1 "PJ301M-12" H 5872 3275 50  0000 R CNN
-F 2 "eurocad:PJ301M-12" H 6350 3200 50  0001 C CNN
+F 2 "eurorack:PJ301M-12" H 6350 3200 50  0001 C CNN
 F 3 "" H 6350 3200 50  0000 C CNN
 	1    6350 3200
@@
 F 0 "U1" H 4458 5796 50  0000 L CNN
 F 1 "TL074" H 4458 5705 50  0000 L CNN
-F 2 "Package_DIP:DIP-14_W8.89mm_SMDSocket_LongPads" H 4450 5850 50  0001 C CNN
+F 2 "Package_DIP:SMDIP-14_W9.53mm" H 4450 5850 50  0001 C CNN
 F 3 "http://www.ti.com/lit/ds/symlink/tl071.pdf" H 4550 5950 50  0001 C CNN
 	5    4500 5750
@@
 F 0 "U3" H 8300 2467 50  0000 C CNN
 F 1 "TL074" H 8300 2376 50  0000 C CNN
-F 2 "Package_DIP:DIP-14_W8.89mm_SMDSocket_LongPads" H 8250 2200 50  0001 C CNN
+F 2 "Package_DIP:SMDIP-14_W9.53mm" H 8250 2200 50  0001 C CNN
 F 3 "http://www.ti.com/lit/ds/symlink/tl071.pdf" H 8350 2300 50  0001 C CNN
 	1    8300 2100
@@
 F 0 "U3" H 8300 2967 50  0000 C CNN
 F 1 "TL074" H 8300 2876 50  0000 C CNN
-F 2 "Package_DIP:DIP-14_W8.89mm_SMDSocket_LongPads" H 8250 2700 50  0001 C CNN
+F 2 "Package_DIP:SMDIP-14_W9.53mm" H 8250 2700 50  0001 C CNN
 F 3 "http://www.ti.com/lit/ds/symlink/tl071.pdf" H 8350 2800 50  0001 C CNN
 	2    8300 2600
@@
 F 0 "U3" H 8300 3467 50  0000 C CNN
 F 1 "TL074" H 8300 3376 50  0000 C CNN
-F 2 "Package_DIP:DIP-14_W8.89mm_SMDSocket_LongPads" H 8250 3200 50  0001 C CNN
+F 2 "Package_DIP:SMDIP-14_W9.53mm" H 8250 3200 50  0001 C CNN
 F 3 "http://www.ti.com/lit/ds/symlink/tl071.pdf" H 8350 3300 50  0001 C CNN
 	3    8300 3100
@@
 F 0 "U3" H 8300 3967 50  0000 C CNN
 F 1 "TL074" H 8300 3876 50  0000 C CNN
-F 2 "Package_DIP:DIP-14_W8.89mm_SMDSocket_LongPads" H 8250 3700 50  0001 C CNN
+F 2 "Package_DIP:SMDIP-14_W9.53mm" H 8250 3700 50  0001 C CNN
 F 3 "http://www.ti.com/lit/ds/symlink/tl071.pdf" H 8350 3800 50  0001 C CNN
 	4    8300 3600
@@
 Connection ~ 7950 2000
 $Comp
-L eurocad:PJ301M-12 J9
+L MLT-rescue:PJ301M-12-eurocad J9
 U 1 1 5CDD3CE2
 P 7600 3400
 F 0 "J9" V 7654 3638 50  0000 L CNN
 F 1 "PJ301M-12" V 7563 3638 50  0000 L CNN
-F 2 "eurocad:PJ301M-12" H 7600 3400 50  0001 C CNN
+F 2 "eurorack:PJ301M-12" H 7600 3400 50  0001 C CNN
 F 3 "" H 7600 3400 50  0000 C CNN
 	1    7600 3400
@@
 Connection ~ 8600 3100
 $Comp
-L eurocad:PJ301M-12 J10
+L MLT-rescue:PJ301M-12-eurocad J10
 U 1 1 5CDD3D17
 P 9350 2200
 F 0 "J10" H 8872 2184 50  0000 R CNN
 F 1 "PJ301M-12" H 8872 2275 50  0000 R CNN
-F 2 "eurocad:PJ301M-12" H 9350 2200 50  0001 C CNN
+F 2 "eurorack:PJ301M-12" H 9350 2200 50  0001 C CNN
 F 3 "" H 9350 2200 50  0000 C CNN
 	1    9350 2200
@@
 $EndComp
 $Comp
-L eurocad:PJ301M-12 J11
+L MLT-rescue:PJ301M-12-eurocad J11
 U 1 1 5CDD3D1D
 P 9350 2700
 F 0 "J11" H 8872 2684 50  0000 R CNN
 F 1 "PJ301M-12" H 8872 2775 50  0000 R CNN
-F 2 "eurocad:PJ301M-12" H 9350 2700 50  0001 C CNN
+F 2 "eurorack:PJ301M-12" H 9350 2700 50  0001 C CNN
 F 3 "" H 9350 2700 50  0000 C CNN
 	1    9350 2700
@@
 $EndComp
 $Comp
-L eurocad:PJ301M-12 J12
+L MLT-rescue:PJ301M-12-eurocad J12
 U 1 1 5CDD3D23
 P 9350 3200
 F 0 "J12" H 8872 3184 50  0000 R CNN
 F 1 "PJ301M-12" H 8872 3275 50  0000 R CNN
-F 2 "eurocad:PJ301M-12" H 9350 3200 50  0001 C CNN
+F 2 "eurorack:PJ301M-12" H 9350 3200 50  0001 C CNN
 F 3 "" H 9350 3200 50  0000 C CNN
 	1    9350 3200
@@
 F 0 "U3" H 4958 5796 50  0000 L CNN
 F 1 "TL074" H 4958 5705 50  0000 L CNN
-F 2 "Package_DIP:DIP-14_W8.89mm_SMDSocket_LongPads" H 4950 5850 50  0001 C CNN
+F 2 "Package_DIP:SMDIP-14_W9.53mm" H 4950 5850 50  0001 C CNN
 F 3 "http://www.ti.com/lit/ds/symlink/tl071.pdf" H 5050 5950 50  0001 C CNN
 	5    5000 5750
@@
 F 0 "U2" H 4708 5796 50  0000 L CNN
 F 1 "TL074" H 4708 5705 50  0000 L CNN
-F 2 "Package_DIP:DIP-14_W8.89mm_SMDSocket_LongPads" H 4700 5850 50  0001 C CNN
+F 2 "Package_DIP:SMDIP-14_W9.53mm" H 4700 5850 50  0001 C CNN
 F 3 "http://www.ti.com/lit/ds/symlink/tl071.pdf" H 4800 5950 50  0001 C CNN
 	5    4750 5750
