File: maske - VCF/maske - VCF.sch (KiCad schematic (older format))
At the start: 183 parts, among them IC1 NE5532, IC100 TL074P, IC101 TL074P, IC2 NE5532, IC3 LM13700N, Q1 2SC1623, Q10 2N3906, Q2 2SC1623, Q3 2SC1623, Q4 2SC1623, Q5 2SC1623, Q6 2SC1623, Q7 2N3819, Q8 2N3819, Q9 2N3906, T1 2N3906, T100 2N3906, T101 2N3906, T2 2N3906

Commit message: mm
Parts:
- removed AUDIO_IN_1, AUDIO_IN_2, AUDIO_OUT_1, AUDIO_OUT_2, CV_IN_CUTOFF_1, CV_IN_CUTOFF_2, CV_IN_CUTOFF_ATT_1, CV_IN_CUTOFF_ATT_2, RES_CV_IN_1, RES_CV_IN_2: WQP-PJ301BM, maske - VCF:WQP-PJ301BM, symbol maske_-_VCF-eagle-import:WQP-PJ301BM
- removed C1, C100, C101, C104, C105, C106, C107, C15, C16, C17, C18, C2, C21, C24: 100n, maske - VCF:C050-025X075, symbol maske_-_VCF-eagle-import:C-EU050-025X075
- removed C10, C102, C103, C22, C25, C9: 1nF poliester, maske - VCF:C050-025X075, symbol maske_-_VCF-eagle-import:C-EU050-025X075
- removed C11, C12: 220uF, maske - VCF:E2,5-7, symbol maske_-_VCF-eagle-import:CPOL-EUE2.5-7
- removed C13, C14: 33uF audio, maske - VCF:E2,5-6, symbol maske_-_VCF-eagle-import:CPOL-EUE2.5-6
- removed C19, C20, C23, C26: 220pF, maske - VCF:C050-025X075, symbol maske_-_VCF-eagle-import:C-EU050-025X075
- removed C3, C4: 10uF, maske - VCF:E2-4, symbol maske_-_VCF-eagle-import:CPOL-EUE2-4
- removed C5, C6: 3.3nF poliester, maske - VCF:C050-025X075, symbol maske_-_VCF-eagle-import:C-EU050-025X075
- removed C7, C8: 10uF, maske - VCF:E2,5-5, symbol maske_-_VCF-eagle-import:CPOL-EUE2.5-5
- removed CUTOFF_A, CUTOFF_ATT_A, CUTOFF_ATT_B, CUTOFF_B, RES_INIT_A, RES_INIT_B, VOL_IN_1, VOL_IN_2: R1212NPADS_GRANDES, maske - VCF:R121N, symbol maske_-_VCF-eagle-import:R1212NPADS_GRANDES
- removed CUTOFF_INIT_A, CUTOFF_INIT_B: 100k, maske - VCF:RTRIM64X, symbol maske_-_VCF-eagle-import:R-TRIMM64X
- removed D1, D2, D5, D6, D7, D8: 1N4148-2, maske - VCF:DO35-2, symbol maske_-_VCF-eagle-import:1N4148-2
- removed D3, D4: 1N5817, maske - VCF:DO35-7, symbol maske_-_VCF-eagle-import:SCHOTTKY-DIODEDO35-7
- removed FERRITE+, FERRITE-: self, maske - VCF:0204_5, symbol maske_-_VCF-eagle-import:R-EU_0204_5
- removed IC1, IC2: NE5532, maske - VCF:DIL08, symbol maske_-_VCF-eagle-import:TL072P
- removed IC100, IC101: TL074P, maske - VCF:DIL14, symbol maske_-_VCF-eagle-import:TL074P
- removed IC3: LM13700N, maske - VCF:DIL16, symbol maske_-_VCF-eagle-import:LM13700N
- removed LED1, LED2: LED3MM, maske - VCF:LED3MM, symbol maske_-_VCF-eagle-import:LED3MM
- removed LINK, LO-HI_SELECT_1, LO-HI_SELECT_2: M9040P, maske - VCF:M9040P, symbol maske_-_VCF-eagle-import:M9040P
- removed LOGO100: OSHW_LOGO_FILLX0200-NT, maske - VCF:OSHW_FILLX200_NOTEXT, symbol maske_-_VCF-eagle-import:OSHW_LOGO_FILLX0200-NT
- removed POWER_IN: IDC_2X5_Acodado, maske - VCF:2X5-RAF, symbol maske_-_VCF-eagle-import:M05X2RAF
- removed Q1, Q2, Q3, Q4, Q5, Q6: 2SC1623, maske - VCF:SOT-23, symbol maske_-_VCF-eagle-import:2SC1623
- removed Q10, Q9, T1, T100, T101, T2: 2N3906, maske - VCF:TO92-EBC, symbol maske_-_VCF-eagle-import:-PNP-TO92-EBC
- removed Q7, Q8: 2N3819, maske - VCF:TO92F, symbol maske_-_VCF-eagle-import:2N3819
- removed R1, R2, R25, R26: 47 Ohm, maske - VCF:0204_5, symbol maske_-_VCF-eagle-import:R-EU_0204_5
- removed R10, R130, R131, R7: 47k, maske - VCF:0204_5, symbol maske_-_VCF-eagle-import:R-EU_0204_5
- removed R100, R101, R102, R103: 1k, maske - VCF:0204_5, symbol maske_-_VCF-eagle-import:R-EU_0204_5
- removed R104, R105, R108, R109, R110, R111, R112, R113, R114, R115, R122, R123, R126, R127, R132, R133: 100k, maske - VCF:0204_5, symbol maske_-_VCF-eagle-import:R-EU_0204_5
- removed R106, R107: 43k, maske - VCF:0204_5, symbol maske_-_VCF-eagle-import:R-EU_0204_5
- removed R11, R12, R43, R44: 4.7k, maske - VCF:0204_5, symbol maske_-_VCF-eagle-import:R-EU_0204_5
- removed R116, R119, R33, R34: 15k, maske - VCF:0204_5, symbol maske_-_VCF-eagle-import:R-EU_0204_5
- removed R117, R118, R120, R121, R124, R125, R128, R129, R13, R14, R17, R18, R21, R22, R23, R24, R8, R9: 10k, maske - VCF:0204_5, symbol maske_-_VCF-eagle-import:R-EU_0204_5
- removed R15, R16: 910k, maske - VCF:0204_5, symbol maske_-_VCF-eagle-import:R-EU_0204_5
- removed R19, R20: 270k, maske - VCF:0204_5, symbol maske_-_VCF-eagle-import:R-EU_0204_5
- removed R27, R28: 820 Ohm, maske - VCF:0204_5, symbol maske_-_VCF-eagle-import:R-EU_0204_5
- removed R29, R30: 33k, maske - VCF:0204_5, symbol maske_-_VCF-eagle-import:R-EU_0204_5
- removed R3, R39, R4, R40: 220 Ohm, maske - VCF:0204_5, symbol maske_-_VCF-eagle-import:R-EU_0204_5
- removed R31, R32: 680 Ohm, maske - VCF:0204_5, symbol maske_-_VCF-eagle-import:R-EU_0204_5
- removed R35, R38: 7.3k, maske - VCF:0204_5, symbol maske_-_VCF-eagle-import:R-EU_0204_5
- removed R36, R37, R51, R52: 3k, maske - VCF:0204_5, symbol maske_-_VCF-eagle-import:R-EU_0204_5
- removed R41, R42: 470 Ohm, maske - VCF:0204_5, symbol maske_-_VCF-eagle-import:R-EU_0204_5
- removed R45, R46: 82k, maske - VCF:0204_5, symbol maske_-_VCF-eagle-import:R-EU_0204_5
- removed R47, R49: 5.6k, maske - VCF:0204_5, symbol maske_-_VCF-eagle-import:R-EU_0204_5
- removed R48, R50: 27k, maske - VCF:0204_5, symbol maske_-_VCF-eagle-import:R-EU_0204_5
- removed R5, R6: 470k, maske - VCF:0204_5, symbol maske_-_VCF-eagle-import:R-EU_0204_5
- removed SV1, SV2: MA05-2T, maske - VCF:MA05-2, symbol maske_-_VCF-eagle-import:MA05-2T
- removed SV3, SV4, SV5, SV6: MA03-2, maske - VCF:MA03-2, symbol maske_-_VCF-eagle-import:MA03-2
- removed U$100: LOGOBEFACOCONLETRAS, maske - VCF:LOGOBEFACOCONLETRAS, symbol maske_-_VCF-eagle-import:LOGOBEFACOCONLETRAS
- added C? (x2): CP1_Small, symbol Device:CP1_Small
- added D?: 1N914, Diode_THT:D_DO-35_SOD27_P7.62mm_Horizontal, symbol Diode:1N914
- added Q? (x3): 2N3904, digikey-footprints:TO-92-3, symbol dk_Transistors-Bipolar-BJT-Single:2N3904
- added R?: R_US, symbol Device:R_US
- added R? (x2): 33k, symbol Device:R_US
- added R? (x6): 100k, symbol Device:R_US
- added R? (x2): 10k, symbol Device:R_US
- added R?: 1m, symbol Device:R_US
- added RV?: R_POT_US, symbol Device:R_POT_US
- added RV? (x2): 100k, symbol Device:R_POT_US
- added RV?: 100, symbol Device:R_POT_US
- added U? (x5): LM13700, symbol Amplifier_Operational:LM13700
- added U? (x5): TL074, symbol Amplifier_Operational:TL074
- added U? (x6): TL072, symbol Amplifier_Operational:TL072
Connections:
- net GND: now also Q?.3 (B), R?.1, U?.3 (+), U?.5 (+)
- new net: R?.1, R?.1, R?.1, R?.1, R?.2, U?.2 (-)
- new net: R?.1, RV?.1, U?.1
- new net: C?.2, Q?.2 (C), R?.1, U?.6 (-)
- new net: C?.1, R?.2, RV?.1, RV?.2, U?.7
- new net: D?.2 (A), Q?.3 (B), RV?.2
- new net: R?.2, RV?.3
- new net: D?.1 (K), R?.2
- new net: R?.1, RV?.3
- new net: Q?.1 (E), Q?.1 (E), R?.1
- new net +12V: R?.1, R?.2, U?.8 (V+)
- new net -12V: R?.1, U?.4 (V-)
- new net CO1: R?.2, RV?.1
- new net CO2: R?.2, RV?.2
- new net CO3: R?.2, RV?.3
- new net CV1: R?.2
- new net CV2: R?.2
- new net CV3: R?.2
Other:
- note removed: "+6V<-->-6V"
- note removed: "-30mV<-->-250mV"
- note removed: "0.28V-p--->"
- note removed: "10mV-p--->"
- note removed: "Peak"
- note removed: "hi_pass_in_1"
- note removed: "lo_pass_in_1"
- note removed: "out_1"
- note removed: "res=max"
- note removed: "res_cv_1"
- note removed: "sine="

Commit message: m
Parts:
- added C? (x2): 220pf, symbol Device:CP1_Small
- added C? (x5): 0.1uf, symbol Device:CP1_Small
- added C?: 22pf, symbol Device:CP1_Small
- added D?: 1N914, Diode_THT:D_DO-35_SOD27_P7.62mm_Horizontal, symbol Diode:1N914
- added J? (x5): PJ301M-12, symbol Eurorack:PJ301M-12
- added Q? (x3): 2N3906, digikey-footprints:TO-92-3, symbol dk_Transistors-Bipolar-BJT-Single:2N3906
- added R? (x2): 7.5k, symbol Device:R_US
- added R? (x2): 20k, symbol Device:R_US
- added R? (x4): 100k, symbol Device:R_US
- added R? (x2): 100, symbol Device:R_US
- added R? (x2): 150k, symbol Device:R_US
- added R?: 43k, symbol Device:R_US
- added R?: 39k, symbol Device:R_US
- added R? (x3): 1m, symbol Device:R_US
- added R? (x2): 2k, symbol Device:R_US
- added R?: 3k, symbol Device:R_US
- added R?: 49.9k, symbol Device:R_US
- added R?: 180k, symbol Device:R_US
- added R?: 4.7m, symbol Device:R_US
- added RV? (x3): 100k, symbol Device:R_POT_US
- added U? (x5): LM13700, symbol Amplifier_Operational:LM13700
- added U? (x3): TL072, symbol Amplifier_Operational:TL072
- added U? (x5): TL074, symbol Amplifier_Operational:TL074
- C?: value CP1_Small -> 100pf
Connections:
- net +12V: now also R?.2, R?.2, U?.11 (V+), U?.4 (V+), U?.8 (V+)
- net -12V: now also R?.1, R?.1, U?.11 (V-), U?.4 (V-), U?.6 (V-)
- net GND: now also C?.2, C?.2, J?.1, J?.1, J?.1, J?.1, J?.1, J?.2, J?.2, J?.2, J?.2, J?.2, Q?.1 (E), Q?.1 (E), R?.1, R?.1, R?.1, R?.2, RV?.1, RV?.1, RV?.1, U?.14 (+), U?.3 (+), U?.3 (+)
- net at Q?.2 (C): now also Q?.2 (B), Q?.2 (B)
- new net: Q?.3 (C), R?.1
- new net: Q?.3 (C), R?.2
- new net: R?.1, U?.1
- new net: R?.1, U?.2 (DIODE_BIAS)
- new net: R?.1, R?.2, R?.2, R?.2, U?.4 (-)
- new net: C?.1, U?.3 (+), U?.5
- new net: C?.1, U?.12, U?.5 (+)
- new net: R?.1, R?.1, R?.2, R?.2, R?.2, U?.13 (-)
- new net: R?.1, U?.15 (DIODE_BIAS)
- new net: R?.2, U?.16
- new net: C?.2, R?.1, R?.1, U?.1, U?.2 (-)
- new net: C?.1, R?.1, R?.2, U?.6 (-), U?.7
- new net: R?.1, R?.1, R?.2, U?.1
- new net: C?.2, R?.2, U?.5 (+)
- new net: R?.1, R?.1, R?.1, R?.2, R?.2, U?.2 (-)
- new net: C?.2, R?.1, R?.2, U?.6 (-)
- new net: C?.1, R?.1, R?.2, U?.7
- new net: C?.1, R?.2 (x3)
- new net: C?.2, RV?.2 (x3)
- new net: J?.3, RV?.3 (x3)
- new net: J?.3, R?.2
- new net: J?.3, R?.1
- new net RB: R?.2
Other:
- moved on the sheet: C?, Q?, R?, RV?, U?A, U?B, U?C, U?D, U?E

Commit message: m
Parts:
- added J?: PJ301M-12, symbol Eurorack:PJ301M-12
- added R?: 2k, symbol Device:R_US
- added R? (x2): 150k, symbol Device:R_US
- added R?: 39k, symbol Device:R_US
- added R?: 4.7m, symbol Device:R_US
- added R?: 49.9, symbol Device:R_US
Connections:
- net GND: now also U?.12 (+), J?.1, J?.2, R?.1, R?.2
- net at C?.1: now also U?.10 (+), R?.2
- net at C?.1, R?.1, R?.2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: now also R?.2
- net at U?.8: now also R?.1, R?.2
- net at U?.9 (-): now also R?.1, R?.2
- net at U?.13 (-): now also R?.1, R?.2
- net RA: now reaches U?.14
- net RA: now also R?.1
- new net: J?.3, R?.1
Other:
- moved on the sheet: U?C, U?D
Changed lines of the file:
@@
 L Amplifier_Operational:TL074 U?
 U 3 1 5D226A27
-P 9400 5400
-F 0 "U?" H 9400 5767 50  0000 C CNN
-F 1 "TL074" H 9400 5676 50  0000 C CNN
-F 2 "" H 9350 5500 50  0001 C CNN
-F 3 "http://www.ti.com/lit/ds/symlink/tl071.pdf" H 9450 5600 50  0001 C CNN
-	3    9400 5400
+P 7500 3550
+F 0 "U?" H 7500 3917 50  0000 C CNN
+F 1 "TL074" H 7500 3826 50  0000 C CNN
+F 2 "" H 7450 3650 50  0001 C CNN
+F 3 "http://www.ti.com/lit/ds/symlink/tl071.pdf" H 7550 3750 50  0001 C CNN
+	3    7500 3550
 	1    0    0    -1
 $EndComp
@@
 L Amplifier_Operational:TL074 U?
 U 4 1 5D226A2D
-P 10950 5400
-F 0 "U?" H 10950 5767 50  0000 C CNN
-F 1 "TL074" H 10950 5676 50  0000 C CNN
-F 2 "" H 10900 5500 50  0001 C CNN
-F 3 "http://www.ti.com/lit/ds/symlink/tl071.pdf" H 11000 5600 50  0001 C CNN
-	4    10950 5400
+P 9400 3550
+F 0 "U?" H 9400 3917 50  0000 C CNN
+F 1 "TL074" H 9400 3826 50  0000 C CNN
+F 2 "" H 9350 3650 50  0001 C CNN
+F 3 "http://www.ti.com/lit/ds/symlink/tl071.pdf" H 9450 3750 50  0001 C CNN
+	4    9400 3550
 	1    0    0    -1
 $EndComp
@@
 	5000 2900 5000 3500
 Connection ~ 5000 3500
+$Comp
+L Device:R_US R?
+U 1 1 5D61A51A
+P 8050 3550
+F 0 "R?" V 7845 3550 50  0000 C CNN
+F 1 "2k" V 7936 3550 50  0000 C CNN
+F 2 "" V 8090 3540 50  0001 C CNN
+F 3 "~" H 8050 3550 50  0001 C CNN
+	1    8050 3550
+	0    1    1    0
+$EndComp
+$Comp
+L Device:R_US R?
+U 1 1 5D61B162
+P 7500 3850
+F 0 "R?" V 7295 3850 50  0000 C CNN
+F 1 "150k" V 7386 3850 50  0000 C CNN
+F 2 "" V 7540 3840 50  0001 C CNN
+F 3 "~" H 7500 3850 50  0001 C CNN
+	1    7500 3850
+	0    1    1    0
+$EndComp
+$Comp
+L Device:R_US R?
+U 1 1 5D61BD45
+P 6950 3850
+F 0 "R?" V 6745 3850 50  0000 C CNN
+F 1 "39k" V 6836 3850 50  0000 C CNN
+F 2 "" V 6990 3840 50  0001 C CNN
+F 3 "~" H 6950 3850 50  0001 C CNN
+	1    6950 3850
+	0    1    1    0
+$EndComp
+$Comp
+L Device:R_US R?
+U 1 1 5D61C559
+P 6750 3650
+F 0 "R?" V 6545 3650 50  0000 C CNN
+F 1 "4.7m" V 6636 3650 50  0000 C CNN
+F 2 "" V 6790 3640 50  0001 C CNN
+F 3 "~" H 6750 3650 50  0001 C CNN
+	1    6750 3650
+	-1   0    0    1
+$EndComp
+$Comp
+L power:GND #PWR?
+U 1 1 5D61D84A
+P 6750 3900
+F 0 "#PWR?" H 6750 3650 50  0001 C CNN
+F 1 "GND" V 6755 3772 50  0000 R CNN
+F 2 "" H 6750 3900 50  0001 C CNN
+F 3 "" H 6750 3900 50  0001 C CNN
+	1    6750 3900
+	1    0    0    -1
+$EndComp
+Wire Wire Line
+	7200 3650 7200 3850
+Wire Wire Line
+	7200 3850 7350 3850
+Wire Wire Line
+	7650 3850 7800 3850
+Wire Wire Line
+	7800 3850 7800 3550
+Wire Wire Line
+	7900 3550 7800 3550
+Connection ~ 7800 3550
+Wire Wire Line
+	7100 3850 7200 3850
+Connection ~ 7200 3850
+Wire Wire Line
+	6750 3900 6750 3850
+Wire Wire Line
+	6750 3850 6800 3850
+Connection ~ 6750 3850
+Wire Wire Line
+	6750 3850 6750 3800
+Wire Wire Line
+	6750 3500 6750 3450
+Wire Wire Line
+	6750 3450 7200 3450
+Wire Wire Line
+	9550 2450 9550 3200
+Wire Wire Line
+	9550 3200 6750 3200
+Wire Wire Line
+	6750 3200 6750 3450
+Connection ~ 6750 3450
+$Comp
+L Eurorack:PJ301M-12 J?
+U 1 1 5D6A4FB0
+P 8100 4400
+F 0 "J?" V 8154 4222 50  0000 R CNN
+F 1 "PJ301M-12" V 8063 4222 50  0000 R CNN
+F 2 "" H 8100 4400 50  0000 C CNN
+F 3 "" H 8100 4400 50  0000 C CNN
+	1    8100 4400
+	0    -1   -1   0
+$EndComp
+Wire Wire Line
+	8200 3950 8200 3550
+Wire Wire Line
+	8100 3950 7950 3950
+$Comp
+L power:GND #PWR?
+U 1 1 5D6A4FB8
+P 8100 3950
+F 0 "#PWR?" H 8100 3700 50  0001 C CNN
+F 1 "GND" V 8105 3822 50  0000 R CNN
+F 2 "" H 8100 3950 50  0001 C CNN
+F 3 "" H 8100 3950 50  0001 C CNN
+	1    8100 3950
+	-1   0    0    1
+$EndComp
+Connection ~ 8100 3950
+$Comp
+L Device:R_US R?
+U 1 1 5D762819
+P 9400 3800
+F 0 "R?" V 9195 3800 50  0000 C CNN
+F 1 "150k" V 9286 3800 50  0000 C CNN
+F 2 "" V 9440 3790 50  0001 C CNN
+F 3 "~" H 9400 3800 50  0001 C CNN
+	1    9400 3800
+	0    1    1    0
+$EndComp
+$Comp
+L Device:R_US R?
+U 1 1 5D763BE6
+P 8850 3650
+F 0 "R?" V 8645 3650 50  0000 C CNN
+F 1 "49.9" V 8736 3650 50  0000 C CNN
+F 2 "" V 8890 3640 50  0001 C CNN
+F 3 "~" H 8850 3650 50  0001 C CNN
+	1    8850 3650
+	0    1    1    0
+$EndComp
+$Comp
+L power:GND #PWR?
+U 1 1 5D764FFF
+P 9100 3450
+F 0 "#PWR?" H 9100 3200 50  0001 C CNN
+F 1 "GND" V 9105 3322 50  0000 R CNN
+F 2 "" H 9100 3450 50  0001 C CNN
+F 3 "" H 9100 3450 50  0001 C CNN
+	1    9100 3450
+	0    1    1    0
+$EndComp
+Wire Wire Line
+	9100 3650 9100 3800
+Wire Wire Line
+	9100 3800 9250 3800
+Wire Wire Line
+	9550 3800 9700 3800
+Wire Wire Line
+	9700 3800 9700 3550
+Wire Wire Line
+	9000 3650 9100 3650
+Connection ~ 9100 3650
+Wire Wire Line
+	5900 3600 5900 3300
+Wire Wire Line
+	5900 3300 8700 3300
+Wire Wire Line
+	8700 3300 8700 3650
+Connection ~ 5900 3600
+Text GLabel 9700 3550 2    50   Input ~ 0
+RA
 $EndSCHEMATC
