File: EnkelMixer/EnkelMixer/EnkelMixer.sch (KiCad schematic (older format))
At the start: 73 parts, among them J1 PJ301M-12, J10 PJ301M-12, J2 PJ301M-12, J3 PJ301M-12, J4 PJ301M-12, J5 PJ301M-12, J6 PJ301M-12, J7 PJ301M-12, J8 PJ301M-12, J9 PJ301M-12, U1 TL074

Commit message: hmm
Parts:
- removed J10, J7, J8: PJ301M-12, eurorack:PJ301M-12, symbol Eurorack:PJ301M-12
- removed R1, R13, R14, R15, R16, R17, R18, R19, R20, R21, R22, R23, R24, R25, R26, R27, R28, R29, R30, R31, R32, R33, R34, R35, R36, R7: 1K, Resistor_THT:R_Axial_DIN0207_L6.3mm_D2.5mm_P5.08mm_Vertical, symbol Device:R_Small_US
- removed RV1, RV10, RV11, RV12, RV13, RV14, RV15, RV16, RV7, RV8, RV9: 10K, Potentiometer_THT:Potentiometer_Alpha_RD901F-40-00D_Single_Vertical, symbol Device:R_POT_US
- added C11, C12: 10pF, Capacitor_THT:C_Disc_D5.0mm_W2.5mm_P5.00mm, symbol Device:CP1_Small
- added D1, D2: D, Diode_THT:D_A-405_P7.62mm_Horizontal, symbol Device:D
- added J2: IN1R, eurorack:PJ301M-12, symbol Eurorack:PJ301M-12
- added J7: EURO_PWR_2x5, Connector_PinHeader_2.54mm:PinHeader_2x05_P2.54mm_Vertical, symbol Eurorack:EURO_PWR_2x5
- added R4, R6: 10K, Resistor_THT:R_Axial_DIN0207_L6.3mm_D2.5mm_P5.08mm_Vertical, symbol Device:R_Small_US
- added RV2: 100K, Potentiometer_THT:Potentiometer_Alpha_RD901F-40-00D_Single_Vertical, symbol Device:R_POT_US
- added RV7: R_POT_Dual_Separate, Potentiometer_THT:Potentiometer_Alpha_RD902F-40-00D_Dual_Vertical, symbol Device:R_POT_Dual_Separate
- C1: value 22pF -> 10pF
- C10, C9: value 0.1uF -> 10uF
- C2: value 0.1uF -> 10pF
- C3, C5, C6, C7, C8: value 0.1uF -> 100nF
- C4: value 22pF -> 100nF
- J1: renamed from J2; value PJ301M-12 -> IN1L
- J3: value PJ301M-12 -> IN2L
- J4: value PJ301M-12 -> IN2R
- J5: value PJ301M-12 -> IN3L
- J6: value PJ301M-12 -> IN3R
- R1: renamed from R4; value 1K -> 10K
- R10, R11, R2, R3, R5, R8, R9: value 1K -> 10K
- R12: value 39K -> 10K
- R7: renamed from R6; value 39K -> 10K
- RV1: renamed from RV2; value 10K -> 100K
- RV3, RV4, RV5, RV6: value 10K -> 100K
- renumbered J1 to J8
Connections:
- net Earth: now also C10.1, C3.2, C4.1, C5.2, C6.1, C7.2, C8.1, C9.2, RV3.1, RV5.1, U1.10 (+), U1.12 (+), J2.1, J7.3 (GND), J7.4 (GND), J7.5 (GND), J7.6 (GND), J7.7 (GND), J7.8 (GND), RV2.1, RV7.3, RV7.6; no longer J1.2, J3.2, J4.2, J5.2, J6.2, J8.2, J9.2, RV3.2, RV5.2
- net Left: now also R1.1, R3.1, R5.1; no longer R2.1, R8.1
- net Right: now also C2.1, R2.1, R8.2, U1.9 (-), R4.1, R6.1; no longer C4.1, R10.1, R12.2, R5.1, U1.6 (-)
- net at C1.2, R7.1, U1.1: now also R9.2; no longer R3.2
- net at U1.8: now also C2.2, R10.2, R8.1
- net at U1.13 (-): now also R10.1, R12.2, C12.1
- net at U1.14: now also R12.1, C12.2, RV7.4
- net -12V: now reaches U1.11 (V-)
- net -12V: now also C10.2, C4.2, C6.2, C8.2, D2.2 (A)
- net +12V: now reaches U1.4 (V+)
- net +12V: now also C3.1, C5.1, C7.1, C9.1, D1.1 (K)
- net Mono1: now reaches J1.3
- net Mono1: now also RV1.3, J2.2; no longer C2.1
- net at R2.2: now also RV2.2
- net at R5.2: now also RV5.2; no longer R1.1
- net Mono2: now reaches J3.3
- net Mono2: now also J4.2, RV3.3; no longer C3.1
- net at RV4.3: now also J4.3; no longer C3.2
- net at RV4.2: now also R4.2; no longer R9.2
- net Mono3: now reaches J5.3
- net Mono3: now also J6.2, RV5.3; no longer C5.1
- net at RV6.3: now also J6.3; no longer C5.2
- net at RV6.2: now also R6.2
- net at J9.3: now also RV7.5; no longer C9.1
- net at J8.3: now also RV7.2; no longer R3.1
- net LeftOut: now reaches R11.1
- net LeftOut: now also U1.7, C11.2, RV7.1; no longer J4.3
- new net: C11.1, R11.2, R9.1, U1.6 (-)
- new net: J2.3, RV2.3
- new net: R3.2, RV3.2
- new net: D1.2 (A), J7.1 (+12V), J7.2 (+12V)
- new net: D2.1 (K), J7.10 (-12V), J7.9 (-12V)
Other:
- moved on the sheet: C1, J8, R1, R7, RV1, U1A, U1B, U1C, U1D, U1E
