File: rør - MLT/MLT.kicad_pcb (KiCad board)
At the start: 2 copper layers, 57.9 x 128.5 mm, 44 parts, among them J1 PJ301M-12, J10 PJ301M-12, J11 PJ301M-12, J12 PJ301M-12, J2 PJ301M-12, J3 PJ301M-12, J4 PJ301M-12, J5 PJ301M-12, J6 PJ301M-12, J7 PJ301M-12, J8 PJ301M-12, J9 PJ301M-12, U1 TL074, U2 TL074, U3 TL074

Commit message: hmm
Parts:
- added D4: LED, LED_THT:LED_D3.0mm_FlatTop, F.Cu at (171.3, 38.1)
- added J10: PJ301M-12, eurorack:PJ301M-12, F.Cu at (165.0, 83.2)
- added J14: PJ301M-12, eurorack:PJ301M-12, F.Cu at (193.5, 83.2)
- added J15: PJ301M-12, eurorack:PJ301M-12, F.Cu at (174.5, 83.2)
- added J16: PJ301M-12, eurorack:PJ301M-12, F.Cu at (184.0, 83.2)
- added R12: 10m, Resistor_SMD:R_0603_1608Metric_Pad1.05x0.95mm_HandSolder, F.Cu at (164.9, 67.3)
- added R14: 1k, Resistor_SMD:R_0603_1608Metric_Pad1.05x0.95mm_HandSolder, F.Cu at (155.2, 60.9)
- added R18: 51, Resistor_SMD:R_0603_1608Metric_Pad1.05x0.95mm_HandSolder, F.Cu at (189.5, 69.8)
- added R19: 51, Resistor_SMD:R_0603_1608Metric_Pad1.05x0.95mm_HandSolder, F.Cu at (176.6, 69.2)
- added R20: 51, Resistor_SMD:R_0603_1608Metric_Pad1.05x0.95mm_HandSolder, F.Cu at (182.5, 69.8)
- added U4: TL074, Package_DIP:SMDIP-14_W9.53mm, F.Cu at (180.2, 54.6)
- J1, J6, J7, J8, J9: footprint eurocad:PJ301M-12 -> eurorack:PJ301M-12
- J11: renamed from J10; footprint eurocad:PJ301M-12 -> eurorack:PJ301M-12
- J12: renamed from J11; footprint eurocad:PJ301M-12 -> eurorack:PJ301M-12
- J13: renamed from J12; footprint eurocad:PJ301M-12 -> eurorack:PJ301M-12
- J2: renamed from J5; footprint eurocad:PJ301M-12 -> eurorack:PJ301M-12
- J3: renamed from J2; footprint eurocad:PJ301M-12 -> eurorack:PJ301M-12
- J4: renamed from J3; footprint eurocad:PJ301M-12 -> eurorack:PJ301M-12
- J5: renamed from J4; footprint eurocad:PJ301M-12 -> eurorack:PJ301M-12
- U1, U2, U3: footprint Package_DIP:DIP-14_W7.62mm -> Package_DIP:SMDIP-14_W9.53mm
- moved C4 21.9 mm to (108.6, 61.1)
- moved C7 21.9 mm to (99.7, 52.8)
- moved C8 21.9 mm to (108.6, 52.8)
- moved J11 21.9 mm to (78.0, 119.3)
- moved R5 21.9 mm to (73.2, 46.0)
- moved R7 21.9 mm to (65.8, 69.5)
- moved R9 21.9 mm to (65.8, 99.9)
- moved U1 21.9 mm to (66.0, 35.3)
- moved C2 21.9 mm to (108.6, 57.9)
- moved J13 21.9 mm to (78.0, 132.0)
- moved J4 21.9 mm to (77.7, 63.2)
- moved J5 21.9 mm to (69.0, 63.2)
- moved R16 21.9 mm to (72.4, 129.0)
- moved R17 21.9 mm to (74.7, 129.0)
- moved C3 21.9 mm to (100.1, 61.1)
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- renumbered D5 to D3, D3 to D5, D4 to D6, R12 to R13, R13 to R15, R14 to R16, R15 to R17, R6 to R2, R2 to R3, R7 to R4, R3 to R5, R4 to R6, R5 to R7
Other:
- board size 57.9 x 128.5 mm -> 19 x 90.8 mm
