File: takt - CLK/ex/takt-exp.sch (KiCad schematic (older format))
At the start: 55 parts, among them J1 PJ301M-12, J2 PJ301M-12, J3 PJ301M-12, J4 PJ301M-12, J5 PJ301M-12, J6 PJ301M-12, J7 PJ301M-12, J8 PJ301M-12, J9 PJ301M-12, Q1 2N3904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

Commit message: update
Connections:
- wire segments 102 -> 99
Changed lines of the file:
@@
 Tr9
-Wire Wire Line
-	1550 3400 1550 3450
-Wire Wire Line
-	4050 3400 4050 3450
-Wire Wire Line
-	6550 3400 6550 3450
 Wire Wire Line
 	1550 3300 1550 3450
