File: takt - CLK/pcb/takt.kicad_pcb (KiCad board)
At the start: 2 copper layers, 39.4 x 106.7 mm, 69 parts, among them J1 PJ301M-12, J2 PJ301M-12, J3 PJ301M-12, J4 PJ301M-12, J5 PJ301M-12, J6 PJ301M-12, J7 PJ301M-12, J8 PJ301M-12, J9 PJ301M-12, Q1 2N3904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

Commit message: update
Parts:
- removed ?: , 
- H2: value POWER -> PIN_HEADER_2x8
Changed lines of the file:
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@@
-(kicad_pcb (version 20171130) (host pcbnew "(5.1.0)-1")
+(kicad_pcb (version 20171130) (host pcbnew "(5.1.2)-1")
   (general
     (thickness 1.6)
@@
     (tracks 518)
     (zones 0)
-    (modules 69)
+    (modules 68)
     (nets 67)
   )
   (page A4)
   (layers
-    (0 F.Cu signal)
-    (31 B.Cu signal)
+    (0 F.Cu signal hide)
+    (31 B.Cu signal hide)
     (32 B.Adhes user)
     (33 F.Adhes user)
@@
     (add_net Tr9)
   )
-  (module "" (layer F.Cu)
-    (at 102.87 53.975)
-    (fp_text reference "" (at 90.805 74.93) (layer F.SilkS)
-      (effects (font (size 1.27 1.27) (thickness 0.15)))
-    )
-    (fp_text value "" (at 90.805 74.93) (layer F.SilkS)
-      (effects (font (size 1.27 1.27) (thickness 0.15)))
-    )
-    (fp_text user ------ (at 0 -0.635) (layer B.Mask)
-      (effects (font (size 1 1) (thickness 0.25)) (justify mirror))
-    )
-  )
   (module Potentiometer_THT:Potentiometer_Alpha_RD901F-40-00D_Single_Vertical (layer F.Cu)
     (at 90.805 74.93 270)
@@
       (effects (font (size 1 1) (thickness 0.15)) (justify mirror))
     )
-    (fp_text value POWER (at 1.27 3.81) (layer B.Fab)
-      (effects (font (size 1 1) (thickness 0.15)) (justify mirror))
-    )
+    (fp_text value PIN_HEADER_2x8 (at 1.27 3.81) (layer B.Fab)
+      (effects (font (size 1 1) (thickness 0.15)) (justify mirror))
+    )
