File: takt - CLK/pcb/takt.kicad_pcb (KiCad board)
At the start: 2 copper layers, 39.4 x 106.7 mm, 68 parts, among them J1 PJ301M-12, J2 PJ301M-12, J3 PJ301M-12, J4 PJ301M-12, J5 PJ301M-12, J6 PJ301M-12, J7 PJ301M-12, J8 PJ301M-12, J9 PJ301M-12, Q1 2N3904, Q2 2N3904, Q3 2N3904, Q4 2N3904, Q5 2N3904, Q6 2N3904, Q7 2N3904, Q8 2N3904, Q9 2N3904

Commit message: takt pcb: koble bakre kobberflate til GND
Flaten på B.Cu hadde ingen nett, så GND-paden til C3 var ukoblet.
Utdatert fyll er fjernet; fyll på nytt (B) og lag nye gerbers før bestilling.

Co-Authored-By: Claude Opus 5.5 <noreply@anthropic.com>
Routing:
- added copper zone on B.Cu, net GND
- removed copper zone on B.Cu, net (none)
Changed lines of the file:
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@@
     )
   )
-  (zone (net 0) (net_name "") (layer B.Cu) (hatch edge 0.508)
+  (zone (net 5) (net_name GND) (layer B.Cu) (hatch edge 0.508)
     (connect_pads (clearance 0.508))
     (min_thickness 0.254)
