File: takt - CLK/dev/GassTass/GassTass.kicad_pcb (KiCad board)
At the start: 2 copper layers, 36 parts, among them J1 EURO_PWR_2x5, Q1 2N3904, Q2 2N3904, Q3 2N3904, Q4 2N3904, Q5 2N3904, Q6 2N3904, Q7 2N3904, Q8 2N3904, Q9 2N3904, U1 Arduino_Nano_v3.x, U2 ATmega328P-PU

Commit message: Gjør nyere autosave-filer til hovedfiler
- GassTass.kicad_pcb: autosave hadde 121 footprints (matcher skjemaet),
  lagret fil bare 37
- nivå - MXR - main.sch: lagret fil var et tomt ark, autosave hadde hele skjemaet

Co-Authored-By: Claude Opus 5.5 <noreply@anthropic.com>
Parts:
- added D10: LED, LED_THT:LED_D3.0mm_FlatTop, F.Cu at (85.4, -8.83)
- added D11: LED, LED_THT:LED_D3.0mm_FlatTop, F.Cu at (72.5, 4.82)
- added D2: LED, LED_THT:LED_D3.0mm_FlatTop, F.Cu at (66.0, 5.82)
- added D3: LED, LED_THT:LED_D3.0mm_FlatTop, F.Cu at (79.5, -8.83)
- added D4: LED, LED_THT:LED_D3.0mm_FlatTop, F.Cu at (103.0, -33.1)
- added D5: LED, LED_THT:LED_D3.0mm_FlatTop, F.Cu at (72.5, -0.73)
- added D6: LED, LED_THT:LED_D3.0mm_FlatTop, F.Cu at (86.3, -14.6)
- added D7: LED, LED_THT:LED_D3.0mm_FlatTop, F.Cu at (92.8, -21.0)
- added D8: LED, LED_THT:LED_D3.0mm_FlatTop, F.Cu at (103.0, -27.6)
- added D9: LED, LED_THT:LED_D3.0mm_FlatTop, F.Cu at (79.0, -3.28)
- added J10: PJ301M-12, eurorack:PJ301M-12, F.Cu at (88.9, 177.8)
- added J11: PJ301M-12, eurorack:PJ301M-12, F.Cu at (101.6, 177.8)
- added J2: PJ301M-12, eurorack:PJ301M-12, F.Cu at (76.2, 139.7)
- added J4: PJ301M-12, eurorack:PJ301M-12, F.Cu at (88.9, 139.7)
- added J5: PJ301M-12, eurorack:PJ301M-12, F.Cu at (101.6, 139.7)
- added J6: PJ301M-12, eurorack:PJ301M-12, F.Cu at (76.2, 158.8)
- added J7: PJ301M-12, eurorack:PJ301M-12, F.Cu at (88.9, 158.8)
- added J8: PJ301M-12, eurorack:PJ301M-12, F.Cu at (101.6, 158.8)
- added J9: PJ301M-12, eurorack:PJ301M-12, F.Cu at (76.2, 177.8)
- added Q1: 2N3904, Package_TO_SOT_THT:TO-92_Inline, F.Cu at (96.8, -26.3)
- added Q10: 2N3904, Package_TO_SOT_THT:TO-92_Inline, F.Cu at (66.3, -5.28)
- added Q11: 2N3904, Package_TO_SOT_THT:TO-92_Inline, F.Cu at (90.3, -32.1)
- added Q12: 2N3904, Package_TO_SOT_THT:TO-92_Inline, F.Cu at (66.3, 0.51)
- added Q13: 2N3904, Package_TO_SOT_THT:TO-92_Inline, F.Cu at (97.2, -38.4)
- added Q14: 2N3904, Package_TO_SOT_THT:TO-92_Inline, F.Cu at (103.8, -44.2)
- added Q15: 2N3904, Package_TO_SOT_THT:TO-92_Inline, F.Cu at (80.1, -19.9)
- added Q16: 2N3904, Package_TO_SOT_THT:TO-92_Inline, F.Cu at (97.2, -44.2)
- added Q17: 2N3904, Package_TO_SOT_THT:TO-92_Inline, F.Cu at (59.8, -5.28)
- added Q18: 2N3904, Package_TO_SOT_THT:TO-92_Inline, F.Cu at (80.1, -14.1)
- added Q19: 2N3904, Package_TO_SOT_THT:TO-92_Inline, F.Cu at (86.6, -19.9)
- added Q2: 2N3904, Package_TO_SOT_THT:TO-92_Inline, F.Cu at (72.8, -6.04)
- added Q3: 2N3904, Package_TO_SOT_THT:TO-92_Inline, F.Cu at (66.8, -11.8)
- added Q4: 2N3904, Package_TO_SOT_THT:TO-92_Inline, F.Cu at (103.8, -38.4)
- added Q5: 2N3904, Package_TO_SOT_THT:TO-92_Inline, F.Cu at (96.8, -32.1)
- added Q6: 2N3904, Package_TO_SOT_THT:TO-92_Inline, F.Cu at (59.8, 6.30)
- added Q7: 2N3904, Package_TO_SOT_THT:TO-92_Inline, F.Cu at (90.3, -26.3)
- added Q8: 2N3904, Package_TO_SOT_THT:TO-92_Inline, F.Cu at (73.3, -11.8)
- added Q9: 2N3904, Package_TO_SOT_THT:TO-92_Inline, F.Cu at (59.8, 0.51)
- added R10: 1k, Resistor_THT:R_Axial_DIN0207_L6.3mm_D2.5mm_P10.16mm_Horizontal, F.Cu at (76.5, -33.3)
- added R11: 200, Resistor_THT:R_Axial_DIN0207_L6.3mm_D2.5mm_P10.16mm_Horizontal, F.Cu at (46.1, 1.59)
- added R12: 1k, Resistor_THT:R_Axial_DIN0207_L6.3mm_D2.5mm_P10.16mm_Horizontal, F.Cu at (76.5, -29.3)
- added R13: R_US, Resistor_THT:R_Axial_DIN0207_L6.3mm_D2.5mm_P10.16mm_Horizontal, F.Cu at (66.4, -17.1)
- added R14: 10k, Resistor_THT:R_Axial_DIN0207_L6.3mm_D2.5mm_P10.16mm_Horizontal, F.Cu at (76.5, -25.2)
- added R15: 1k, Resistor_THT:R_Axial_DIN0207_L6.3mm_D2.5mm_P10.16mm_Horizontal, F.Cu at (46.1, 5.64)
- added R16: 1k, Resistor_THT:R_Axial_DIN0207_L6.3mm_D2.5mm_P10.16mm_Horizontal, F.Cu at (83.5, -41.4)
- added R17: 200, Resistor_THT:R_Axial_DIN0207_L6.3mm_D2.5mm_P10.16mm_Horizontal, F.Cu at (53.1, -10.6)
- added R18: 1k, Resistor_THT:R_Axial_DIN0207_L6.3mm_D2.5mm_P10.16mm_Horizontal, F.Cu at (83.5, -45.5)
- added R19: 10k, Resistor_THT:R_Axial_DIN0207_L6.3mm_D2.5mm_P10.16mm_Horizontal, F.Cu at (63.2, -25.2)
- added R2: 200, Resistor_THT:R_Axial_DIN0207_L6.3mm_D2.5mm_P10.16mm_Horizontal, F.Cu at (19.5, 6.59)
- added R20: 1k, Resistor_THT:R_Axial_DIN0207_L6.3mm_D2.5mm_P10.16mm_Horizontal, F.Cu at (70.2, -45.5)
- added R21: 1k, Resistor_THT:R_Axial_DIN0207_L6.3mm_D2.5mm_P10.16mm_Horizontal, F.Cu at (63.2, -29.3)
- added R22: 200, Resistor_THT:R_Axial_DIN0207_L6.3mm_D2.5mm_P10.16mm_Horizontal, F.Cu at (63.2, -33.3)
- added R23: 1k, Resistor_THT:R_Axial_DIN0207_L6.3mm_D2.5mm_P10.16mm_Horizontal, F.Cu at (70.2, -37.4)
- added R24: 10k, Resistor_THT:R_Axial_DIN0207_L6.3mm_D2.5mm_P10.16mm_Horizontal, F.Cu at (32.8, 0.04)
- added R25: 1k, Resistor_THT:R_Axial_DIN0207_L6.3mm_D2.5mm_P10.16mm_Horizontal, F.Cu at (53.1, -18.7)
- added R26: 1k, Resistor_THT:R_Axial_DIN0207_L6.3mm_D2.5mm_P10.16mm_Horizontal, F.Cu at (39.8, -10.6)
- added R27: 200, Resistor_THT:R_Axial_DIN0207_L6.3mm_D2.5mm_P10.16mm_Horizontal, F.Cu at (32.8, -4.01)
- added R28: 1k, Resistor_THT:R_Axial_DIN0207_L6.3mm_D2.5mm_P10.16mm_Horizontal, F.Cu at (70.2, -41.4)
- added R29: 10k, Resistor_THT:R_Axial_DIN0207_L6.3mm_D2.5mm_P10.16mm_Horizontal, F.Cu at (49.9, -22.7)
- added R30: 1k, Resistor_THT:R_Axial_DIN0207_L6.3mm_D2.5mm_P10.16mm_Horizontal, F.Cu at (26.5, -8.06)
- added R31: 1k, Resistor_THT:R_Axial_DIN0207_L6.3mm_D2.5mm_P10.16mm_Horizontal, F.Cu at (32.8, 4.09)
- added R32: 200, Resistor_THT:R_Axial_DIN0207_L6.3mm_D2.5mm_P10.16mm_Horizontal, F.Cu at (26.5, -16.2)
- added R33: 1k, Resistor_THT:R_Axial_DIN0207_L6.3mm_D2.5mm_P10.16mm_Horizontal, F.Cu at (56.9, -37.4)
- added R34: 10k, Resistor_THT:R_Axial_DIN0207_L6.3mm_D2.5mm_P10.16mm_Horizontal, F.Cu at (19.5, 2.54)
- added R35: 1k, Resistor_THT:R_Axial_DIN0207_L6.3mm_D2.5mm_P10.16mm_Horizontal, F.Cu at (39.8, -18.7)
- added R36: 1k, Resistor_THT:R_Axial_DIN0207_L6.3mm_D2.5mm_P10.16mm_Horizontal, F.Cu at (19.5, -1.51)
- added R37: 200, Resistor_THT:R_Axial_DIN0207_L6.3mm_D2.5mm_P10.16mm_Horizontal, F.Cu at (56.9, -41.4)
- added R38: 1k, Resistor_THT:R_Axial_DIN0207_L6.3mm_D2.5mm_P10.16mm_Horizontal, F.Cu at (6.16, -1.51)
- added R39: 10k, Resistor_THT:R_Axial_DIN0207_L6.3mm_D2.5mm_P10.16mm_Horizontal, F.Cu at (6.16, 2.54)
- added R40: 1k, Resistor_THT:R_Axial_DIN0207_L6.3mm_D2.5mm_P10.16mm_Horizontal, F.Cu at (36.6, -30.8)
- added R41: 1k, Resistor_THT:R_Axial_DIN0207_L6.3mm_D2.5mm_P10.16mm_Horizontal, F.Cu at (83.5, -37.4)
- added R42: 200, Resistor_THT:R_Axial_DIN0207_L6.3mm_D2.5mm_P10.16mm_Horizontal, F.Cu at (36.6, -22.7)
- added R43: 1k, Resistor_THT:R_Axial_DIN0207_L6.3mm_D2.5mm_P10.16mm_Horizontal, F.Cu at (6.16, 6.59)
- added R44: 10k, Resistor_THT:R_Axial_DIN0207_L6.3mm_D2.5mm_P10.16mm_Horizontal, F.Cu at (26.5, -12.1)
- added R45: 1k, Resistor_THT:R_Axial_DIN0207_L6.3mm_D2.5mm_P10.16mm_Horizontal, F.Cu at (56.9, -45.5)
- added R46: 1k, Resistor_THT:R_Axial_DIN0207_L6.3mm_D2.5mm_P10.16mm_Horizontal, F.Cu at (53.1, -14.6)
- added R47: 200, Resistor_THT:R_Axial_DIN0207_L6.3mm_D2.5mm_P10.16mm_Horizontal, F.Cu at (39.8, -14.6)
- added R48: 1k, Resistor_THT:R_Axial_DIN0207_L6.3mm_D2.5mm_P10.16mm_Horizontal, F.Cu at (46.1, -6.51)
- added R49: 10k, Resistor_THT:R_Axial_DIN0207_L6.3mm_D2.5mm_P10.16mm_Horizontal, F.Cu at (32.8, 8.14)
- added R50: 1k, Resistor_THT:R_Axial_DIN0207_L6.3mm_D2.5mm_P10.16mm_Horizontal, F.Cu at (66.4, -21.2)
- added R51: 1k, Resistor_THT:R_Axial_DIN0207_L6.3mm_D2.5mm_P10.16mm_Horizontal, F.Cu at (46.1, -2.46)
- added R7: 1k, Resistor_THT:R_Axial_DIN0207_L6.3mm_D2.5mm_P10.16mm_Horizontal, F.Cu at (49.9, -26.8)
- added R8: 10k, Resistor_THT:R_Axial_DIN0207_L6.3mm_D2.5mm_P10.16mm_Horizontal, F.Cu at (49.9, -30.8)
- added R9: 1k, Resistor_THT:R_Axial_DIN0207_L6.3mm_D2.5mm_P10.16mm_Horizontal, F.Cu at (36.6, -26.8)
- moved R1 104.7 mm to (162.6, 91.4)
- moved U1 38.4 mm to (109.2, 20.3)
- moved U2 37.6 mm to (153.7, 50.8)
- moved D1 37.5 mm to (219.7, 62.2)
Connections:
- U1 pad 10: Net-(D7-Pad2) -> Tr6-in
- U1 pad 11: Net-(D8-Pad2) -> Tr7-in
- U1 pad 12: Net-(D9-Pad2) -> Tr8-in
- U1 pad 13: Net-(D10-Pad2) -> Tr9-in
- U1 pad 5: Net-(D2-Pad2) -> Tr1-in
- U1 pad 6: Net-(D3-Pad2) -> Tr2-in
- U1 pad 7: Net-(D4-Pad2) -> Tr3-in
- U1 pad 8: Net-(D5-Pad2) -> Tr4-in
- U1 pad 9: Net-(D6-Pad2) -> Tr5-in
